File: hardware/eagle_layouts/wireless_lab_monitor-sensor_hardware/Single_Item_Sensor_v2.brd (EAGLE design)
At the start: 48.3 x 30.5 mm, 25 parts, among them IC1 H-E Sensor, M1 NRF24L01SMD, U1 ATMEGA328P-AU, X1 Door Sensor

Commit message: Adding v2 hardware designs
Routing:
- net VCC: track 56.7 -> 161.1 mm, vias 0 -> 6
- net GND: track 50.9 -> 149.2 mm, vias 0 -> 3
- net TEMP_PWR: track 0.00 -> 88.3 mm, vias 0 -> 3
- net RXD: track 0.00 -> 60.9 mm
- net TEMP_DATA: track 36.2 -> 81.2 mm, vias 0 -> 1
- net MOSI: track 9.56 -> 48.8 mm
- net RESET: track 22.7 -> 61.3 mm, vias 0 -> 4
- net SCK: track 0.00 -> 35.4 mm, vias 0 -> 2
- net INT_SENSOR_PORT: track 47.3 -> 79.9 mm, vias 0 -> 3
- net SENSOR_PORT: track 0.00 -> 30.5 mm, vias 0 -> 2
- net TXD: track 7.36 -> 31.3 mm, vias 0 -> 1
- net CSN: track 0.00 -> 20.2 mm, vias 0 -> 2
- net DTR: track 0.00 -> 15.4 mm, vias 0 -> 1
- net MISO: track 10.3 -> 25.2 mm, vias 0 -> 2
- net HB_LED: track 0.00 -> 14.0 mm, vias 0 -> 2
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Other:
- board text added: "GND"
- board text added: "MISO"
- board text added: "Wireless Lab Monitor Sensor v2.0 February 2018"
- board text removed: "Wireless Lab Monitor Sensor v1.0 January 2018"

Commit message: Working version with NodeManager 1.6
Parts:
- removed R6, R7, R8: 4.7k, adafruit:M0805
Connections:
- removed net N$1: M1.4, R6.2
- removed net N$2: M1.3, R7.2
- removed net N$3: M1.2, R8.2
- net MISO: no longer R8.1
- net MOSI: no longer R7.1
- net SCK: no longer R6.1
Routing:
- net GND: track 149.2 -> 222.3 mm, vias 3 -> 2
- net RXD: track 60.9 -> 23.9 mm
- net INT_SENSOR_PORT: track 79.9 -> 54.5 mm
- net MOSI: track 48.8 -> 23.6 mm
- net TEMP_DATA: track 81.2 -> 56.2 mm, vias 1 -> 2
- net VCC: track 161.1 -> 141.6 mm, vias 6 -> 8
- net SCK: track 35.4 -> 18.5 mm, vias 2 -> 0
- net TEMP_PWR: track 88.3 -> 71.9 mm, vias 3 -> 0
- net RESET: track 61.3 -> 54.2 mm, vias 4 -> 5
- net CSN: track 20.2 -> 13.9 mm, vias 2 -> 0
- net N$3: track 4.22 -> 0.00 mm
- net N$1: track 3.70 -> 0.00 mm
- net TXD: track 31.3 -> 34.9 mm
- net N$2: track 2.92 -> 0.00 mm
- net MISO: track 25.2 -> 28.0 mm, vias 2 -> 0
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