File: hardware/eagle_layouts/wireless_lab_monitor-sensor_hardware/Single_Item_Sensor_v2.sch (EAGLE design)
At the start: 25 parts, among them IC1 H-E Sensor, M1 NRF24L01SMD, U1 ATMEGA328P-AU, X1 Door Sensor

Commit message: Working version with NodeManager 1.6
Parts:
- removed R6, R7, R8: 4.7k, adafruit:R-US_M0805
Connections:
- removed net N$1: M1.SCK, R6.2
- removed net N$2: M1.MOSI, R7.2
- removed net N$3: M1.MISO, R8.2
- net MISO: no longer R8.1
- net MOSI: no longer R7.1
- net SCK: no longer R6.1
Changed lines of the file:
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@@
 <part name="C3" library="GDOv5 Board" deviceset="CAP" device="0805" value="0.1uF"/>
 <part name="ISP1" library="adafruit" deviceset="AVRISP" device="-6"/>
-<part name="R6" library="adafruit" deviceset="R-US_" device="M0805" value="4.7k"/>
-<part name="R7" library="adafruit" deviceset="R-US_" device="M0805" value="4.7k"/>
-<part name="R8" library="adafruit" deviceset="R-US_" device="M0805" value="4.7k"/>
 </parts>
 <sheets>
@@
 </instance>
 <instance part="ISP1" gate="G$1" x="142.24" y="-10.16"/>
-<instance part="R6" gate="G$1" x="38.1" y="-12.7" smashed="yes">
-<attribute name="NAME" x="33.274" y="-12.4714" size="1.27" layer="95"/>
-<attribute name="VALUE" x="40.64" y="-14.224" size="1.27" layer="96"/>
-</instance>
-<instance part="R7" gate="G$1" x="38.1" y="-15.24" smashed="yes">
-<attribute name="NAME" x="33.274" y="-15.0114" size="1.27" layer="95"/>
-<attribute name="VALUE" x="40.894" y="-16.764" size="1.27" layer="96"/>
-</instance>
-<instance part="R8" gate="G$1" x="38.1" y="-17.78" smashed="yes">
-<attribute name="NAME" x="33.02" y="-17.5514" size="1.27" layer="95"/>
-<attribute name="VALUE" x="40.64" y="-19.304" size="1.27" layer="96"/>
-</instance>
 </instances>
 <busses>
@@
 </segment>
 <segment>
-<pinref part="R6" gate="G$1" pin="1"/>
-<wire x1="33.02" y1="-12.7" x2="30.48" y2="-12.7" width="0.1524" layer="91"/>
-<label x="30.48" y="-12.7" size="1.016" layer="95" rot="R180" xref="yes"/>
+<wire x1="45.72" y1="-12.7" x2="43.18" y2="-12.7" width="0.1524" layer="91"/>
+<label x="43.18" y="-12.7" size="1.016" layer="95" rot="R180" xref="yes"/>
 </segment>
 <segment>
@@
 </segment>
 <segment>
-<pinref part="R7" gate="G$1" pin="1"/>
-<wire x1="33.02" y1="-15.24" x2="30.48" y2="-15.24" width="0.1524" layer="91"/>
-<label x="30.48" y="-15.24" size="1.016" layer="95" rot="R180" xref="yes"/>
+<wire x1="45.72" y1="-15.24" x2="43.18" y2="-15.24" width="0.1524" layer="91"/>
+<label x="43.18" y="-15.24" size="1.016" layer="95" rot="R180" xref="yes"/>
 </segment>
 <segment>
@@
 </segment>
 <segment>
-<pinref part="R8" gate="G$1" pin="1"/>
-<wire x1="33.02" y1="-17.78" x2="30.48" y2="-17.78" width="0.1524" layer="91"/>
-<label x="30.48" y="-17.78" size="1.016" layer="95" rot="R180" xref="yes"/>
+<wire x1="45.72" y1="-17.78" x2="43.18" y2="-17.78" width="0.1524" layer="91"/>
+<label x="43.18" y="-17.78" size="1.016" layer="95" rot="R180" xref="yes"/>
 </segment>
 <segment>
@@
 </segment>
 </net>
-<net name="N$1" class="0">
-<segment>
-<pinref part="M1" gate="G$1" pin="SCK"/>
-<wire x1="45.72" y1="-12.7" x2="43.18" y2="-12.7" width="0.1524" layer="91"/>
-<pinref part="R6" gate="G$1" pin="2"/>
-</segment>
-</net>
-<net name="N$2" class="0">
-<segment>
-<pinref part="M1" gate="G$1" pin="MOSI"/>
-<wire x1="45.72" y1="-15.24" x2="43.18" y2="-15.24" width="0.1524" layer="91"/>
-<pinref part="R7" gate="G$1" pin="2"/>
-</segment>
-</net>
-<net name="N$3" class="0">
-<segment>
-<pinref part="M1" gate="G$1" pin="MISO"/>
-<wire x1="45.72" y1="-17.78" x2="43.18" y2="-17.78" width="0.1524" layer="91"/>
-<pinref part="R8" gate="G$1" pin="2"/>
-</segment>
-</net>
